Commit message: fix(imu): mount the IMU where it now sits -- yawed -90 deg, off-centre
The IMU moved: it sits upright at xyz 0.053 0 0.012 in base_link,
yawed -90 deg (chip +y forward, +x to the robot's right).

* body.urdf.xacro: imu_joint carries the new pose; also drop the stray
  trailing space in the camera_link name that broke the camera's TF.
* launch_common: one IMU_MOUNT_RPY copy of the URDF rpy, passed to
  policy_node and, new, to leg_odometry_node.
* leg_odometry_node: takes imu_mount_rpy and rotates the IMU orientation
  and gyro into base_link. It read the sensor axes as base axes, which
  under a yawed mount swaps roll/pitch in stance detection and the odom
  pose.
* sim: the MuJoCo plugin emulates the same mount (wojtek_sim.urdf.xacro,
  and the plugin's default), so the sim exercises the compensation the
  robot needs instead of undoing a rotation it never applied.
* mocks keep identity orientation: a pure yaw moves neither gravity nor
  accel z, so it is still a level reading; comments and a test docstring
  now say so.

Not yet validated on hardware: confirm the sign with a tilt test (nose
down -> accel y < 0, right side down -> accel x < 0).

Co-Authored-By: Claude Opus 5.5 <noreply@anthropic.com>

File: ros/src/wojtek_description/urdf/body.urdf.xacro (robot description, xacro)
@@ -41,8 +41,12 @@
     </joint>
     <link name="imu_link" />
-    <!-- The Adafruit 5543 sits UPRIGHT: measured at rest on the robot,
-         linear_acceleration.z = +10.05 m/s2, and imu_i2c.cpp reads the chip
-         axes straight into x/y/z with no remap. The rpy 0 pi 0 that stood
-         here was left over from the previous IMU and made policy_node flip
+    <!-- The Adafruit 5543 sits UPRIGHT (measured at rest on the robot,
+         linear_acceleration.z = +10.05 m/s2) and yawed -90 deg: the chip's
+         +y points forward, its +x to the robot's right. imu_i2c.cpp reads
+         the chip axes straight into x/y/z with no remap, so this rotation
+         is the only place the mount is undone; launch_common's
+         IMU_MOUNT_RPY copies it for policy_node and leg_odometry, and
+         wojtek_sim.urdf.xacro's imu_mount_rpy emulates it. An earlier
+         rpy 0 pi 0 left over from the previous IMU made policy_node flip
          gravity and the gyro's x/z, which stayed invisible until a policy
          actually read the IMU (terrain_blind v41). That one then fought a
@@ -51,5 +55,5 @@
       <parent link="base_link" />
       <child link="imu_link" />
-      <origin xyz="0.0 0.0 0.1" rpy="0.0 0.0 0.0" />
+      <origin xyz="0.053 0.0 0.012" rpy="0.0 0.0 -1.5707963" />
     </joint>
     <xacro:if value="${with_camera}">

Commit message: feat(bringup): the robot's URDF carries the D435 mount; extrinsics.yaml gets the design numbers
The costmap, the pixel resolver and the VLM brain's bearing all transform
camera points into odom, which needs base_link -> camera_link. On the
robot that edge came from wojtek_perception_bringup's extrinsics.yaml,
a placeholder of zeros ("camera in the middle of the body, looking
level"), published only under perception:=true; the deck-camera mode the
service runs published nothing at all. The sim had the real mount all
along (with_camera in body.urdf.xacro), which is why navigation worked
there and could not on the robot.

- body.urdf.xacro: the mount (camera_link + camera_joint, 0.32 m ahead,
  0.07 m up, 15 deg down) is its own macro; with_camera_mount adds just
  that, with_camera (the sim) adds it plus the optical chain. The real
  robot must not carry the optical frames: the realsense2_camera driver
  publishes camera_link -> *_optical itself and two publishers of one
  edge fight.
- wojtek_real.urdf.xacro: with_camera_mount="true", so the
  robot_state_publisher gives the edge in every mode with a camera
  (deck_camera:=true and perception:=true alike).
- launch_common: the perception include gets extrinsics:=false, the
  bringup owns the edge now.
- extrinsics.yaml: the design mount instead of zeros, for a standalone
  perception launch; header says it is the drawing, to be confirmed
  with a tape measure and a floor check on the head.
- Tests: the real URDF renders with the mount at the design pose and
  without the optical frames, also under mock_hw; the yaml agrees with
  the URDF (wojtek_bringup) and with camera_spec (wojtek_pc).

Co-Authored-By: Claude Fable 5.1 <noreply@anthropic.com>
Claude-Session: https://claude.ai/code/session_01T3xdzRKqo85ydjYaBcAhwq

File: ros/src/wojtek_description/urdf/body.urdf.xacro (robot description, xacro)
@@ -7,12 +7,40 @@
        blocks are deliberately not part of this macro - callers add their
        own on top (see wojtek.urdf.xacro for the stock example).
-       with_camera adds the D435 mount frames (camera_link + optical
-       frames). Default OFF: on the real robot the realsense2_camera driver
-       publishes the camera_link->*_optical chain itself and two publishers
-       of the same TF edge fight. The sim URDF turns it on: there the
-       robot model owns the ground-truth extrinsics (machinekind/wojtek#91).
+       The D435 comes in two shapes, both default OFF, never both on:
+         with_camera_mount  base_link -> camera_link only. The real robot:
+                            the realsense2_camera driver publishes the
+                            camera_link -> *_optical chain itself (two
+                            publishers of one TF edge fight), but cannot
+                            know where the camera sits on the body, and the
+                            costmap, the pixel resolver and the VLM brain
+                            need that edge in every mode with a camera.
+         with_camera        the mount and the optical frames. The sim: the
+                            robot model owns the ground-truth extrinsics
+                            (machinekind/wojtek#91).
        The mount numbers must match wojtek_pc/camera_spec.py (MOUNT_XYZ,
-       MOUNT_PITCH_RAD); a test cross-checks them. -->
-  <xacro:macro name="wojtek_body" params="with_camera:=false">
+       MOUNT_PITCH_RAD) and wojtek_perception_bringup/config/extrinsics.yaml;
+       tests cross-check all three. -->
+  <xacro:macro name="camera_mount">
+    <!-- D435 mount: camera_link (x forward, z up, ROS body convention)
+         at the centre of the head bracket (front face of the body mesh's
+         triangular head section), pitched 15 deg down (0.2617994 rad). -->
+    <link name="camera_link">
+      <visual>
+        <!-- Camera-body sized marker so the mount is visible in RViz;
+             massless. -->
+        <origin xyz="-0.01 0 0" rpy="0 0 0" />
+        <geometry>
+          <box size="0.02 0.09 0.025" />
+        </geometry>
+        <xacro:grey_material />
+      </visual>
+    </link>
+    <joint name="camera_joint" type="fixed">
+      <parent link="base_link" />
+      <child link="camera_link" />
+      <origin xyz="0.32 0.0 0.07" rpy="0 0.2617994 0" />
+    </joint>
+  </xacro:macro>
+  <xacro:macro name="wojtek_body" params="with_camera:=false with_camera_mount:=false">
     <material name="grey">
       <color rgba="0.5 0.5 0.5 1" />
@@ -57,29 +85,13 @@
       <origin xyz="0.053 0.0 0.012" rpy="0.0 0.0 -1.5707963" />
     </joint>
+    <xacro:if value="${with_camera_mount}">
+      <xacro:camera_mount />
+    </xacro:if>
     <xacro:if value="${with_camera}">
-      <!-- D435 mount: camera_link (x forward, z up, ROS body convention)
-           at the centre of the head bracket (front face of the body mesh's
-           triangular head section), pitched down; then the standard
-           camera_frame -> optical_frame (z forward, x right, y down)
-           rotation. Frame names follow the realsense2_camera driver
-           (camera_name=camera) so consumers see identical TF in sim and
-           on the robot. Values mirror camera_spec.py: MOUNT_XYZ /
-           MOUNT_PITCH_RAD (15 deg = 0.2617994 rad). -->
-      <link name="camera_link">
-        <visual>
-          <!-- Camera-body sized marker so the mount is visible in RViz;
-               massless. -->
-          <origin xyz="-0.01 0 0" rpy="0 0 0" />
-          <geometry>
-            <box size="0.02 0.09 0.025" />
-          </geometry>
-          <xacro:grey_material />
-        </visual>
-      </link>
-      <joint name="camera_joint" type="fixed">
-        <parent link="base_link" />
-        <child link="camera_link" />
-        <origin xyz="0.32 0.0 0.07" rpy="0 0.2617994 0" />
-      </joint>
+      <!-- The mount, then the standard camera_frame -> optical_frame
+           (z forward, x right, y down) rotation. Frame names follow the
+           realsense2_camera driver (camera_name=camera) so consumers see
+           identical TF in sim and on the robot. -->
+      <xacro:camera_mount />
       <link name="camera_depth_frame" />
       <joint name="camera_depth_joint" type="fixed">
